Commit message: Add files via upload

File: mp500_description/urdf/mp500.urdf.xacro (robot description, xacro)
@@ -6,71 +6,38 @@
   <xacro:property name="safety_offset" value="0.02"/>
 <!-- Materials -->
-    <material name="Neobotix/Black">
-        <color rgba="0.0 0.0 0.0 1.0"/>
-    </material>
-    <material name="Neobotix/Blue">
-        <color rgba="0.0 0.0 0.8 1.0"/>
-    </material>
-    <material name="Neobotix/Green">
-        <color rgba="0.0 0.8 0.0 1.0"/>
-    </material>
-    <material name="Neobotix/Grey">
-        <color rgba="0.7 0.7 0.7 1.0"/>
-    </material>
-    <material name="Neobotix/Grey2">
-        <color rgba="0.9 0.9 0.9 1.0"/>
-    </material>
-    <material name="Neobotix/Red">
-        <color rgba="0.8 0.0 0.0 1.0"/>
-    </material>
-    <material name="Neobotix/White">
-        <color rgba="1.0 1.0 1.0 1.0"/>
-    </material>
-    <material name="Neobotix/Yellow">
-        <color rgba="1.0 1.0 0 10" />
-    </material>
-   <material name="Schunk/LightGrey">
-        <color rgba="0.7 0.7 0.7 1.0"/>
-   </material>
-   <material name="Schunk/DarkGrey">
-        <color rgba="0.4 0.4 0.4 1.0"/>
-   </material>
-   <material name="Schunk/Black">
-        <color rgba="0.0 0.0 0.0 1.0"/>
-   </material>
-   <material name="Schunk/DarkGolden">
-        <color rgba="0.4 0.4 0.3 1.0"/>
-   </material>
-   <material name="Schunk/Blue">
-        <color rgba="0.0 0.0 0.8 1.0"/>
-   </material>
-  <!--neo_mp_500-->
-  <!--xacro:include filename="$(find neo_mp_500)/robot_model/mp_500/mp500.urdf.xacro" /-->
 <!--++++++++++++++++++++++++++++++base_link++++++++++++++++++++++++++++++++++++++++++++++++++++-->
-<!--++++++++++++++++++++body++++++++++++++++++++++++++++-->
   <link name="base_link">
        <inertial>
           <mass value="25.67" />
-	    <origin xyz="0 0 0.216" rpy="0 0 0"/>
-	<inertia ixx="0.54" ixy="0.0" ixz="0.0" iyy="1.08" iyz="0.0" izz="1.23" />
+	    <origin xyz="0.15 0 0.2" rpy="0 0 0"/>
+	<inertia ixx="1.08" ixy="0.0" ixz="0.0" iyy="1.08" iyz="0.0" izz="1.23" />
        </inertial>
        <visual name='body'>
-        <!--origin xyz="0.0 0.0 0.234" rpy="0 0 1.57" /--><!-- for cylinder -->
-	<origin xyz="-0.160 0.0 0.09" rpy="0 0 -1.57" /><!-- for STL -->
+	<origin xyz="0 0 0.09" rpy="0 0 -1.57" /><!-- for STL -->
               <geometry>
-                 <mesh filename="package://neo_mp_500/robot_model/mp_500/meshes/MP500-BODY.STL" scale="0.01 0.01 0.01"/>
-	    	<!--cylinder length="0.381" radius="0.2545"/-->
-	    	<!--box size="0.445 0.277 0.17"/-->
-              </geometry>
+                 <mesh filename="package://mp500_description/meshes/MP500-BODY.STL" scale="0.01 0.01 0.01"/>
+	      </geometry>
         <material name="Neobotix/Grey" />
        </visual>
       <collision name='body_collision'>
-        <origin xyz="0 0 0.216" rpy="0 0 -1.57" />
+        <origin xyz="0.1 0 0.2" rpy="0 0 -1.57" />
         <geometry>
-          <box size="0.400 0.676 0.300"/>
-          <!--cylinder length="0.381" radius="0.2545"/-->
+          <box size="0.400 0.400 0.250"/>
         </geometry>
       </collision>
-   </link>
+      <visual>
+	  <origin xyz="0.45 0 0.01" rpy="0 0 0" />
+	  <geometry>
+            <sphere radius="0.005"/>
+	  </geometry>
+	 <material name="Neobotix/Grey" />
+	</visual>
+        <collision>
+	  <origin xyz="0.45 0 0.01" rpy="0 0 0" />
+	  <geometry>
+             <sphere radius="0.005"/>
+	  </geometry>
+	</collision>
+    </link>
 <!--+++++++++++++++++++wheel_left_link++++++++++++++++++++++++-->
    <link name="wheel_left_link" type="wheel">
@@ -83,5 +50,5 @@
      	<origin xyz="0 0 0" rpy="0 0 -1.57" />
      	<geometry>
-		<mesh filename="package://neo_mp_500/robot_model/mp_500/meshes/MP500-WHEEL.STL" scale="0.01 0.01 0.01" />
+		<mesh filename="package://mp500_description/meshes/MP500-WHEEL.STL" scale="0.01 0.01 0.01" />
      	</geometry>
      	<material name="Neobotix/Black" />
@@ -96,5 +63,5 @@
 <!--+++++++++++++++++++wheel_left_joint++++++++++++++++++++++++-->
   <joint name="wheel_left_joint" type="revolute">
-     <origin xyz="-0.155 0.255 0.13" rpy="0 0 0" />
+     <origin xyz="0 0.255 0.13" rpy="0 0 0" />
     	<axis xyz="0 1 0"/>
     	<limit effort="10000.0" lower="-1e+16" upper="1e+16" velocity="11.6"/>
@@ -104,32 +71,4 @@
     </joint>
 <!--+++++++++++++++++++wheel_right_link++++++++++++++++++++++++-->
-<!--Mesh Volume is 3587.704102
-Mesh Surface is 1876.550415
-Thin shell barycenter -25.340059 -0.000027 4.499997
-Center of Mass is -25.340000 -0.000164 4.500009
-Inertia Tensor is :
-| 322624.937500 -0.068522 -1.293689 |
-| -0.068522 179104.328125 -1.342927 |
-| -1.293689 -1.342927 179079.796875 |
-Principal axes are :
-| 1.000000 -0.000000 0.000009 |
-| -0.000000 0.998514 0.054499 |
-| -0.000009 -0.054499 0.998514 |
-axis momenta are :
-| 322624.937500 179104.406250 179079.718750 |
-Mesh Volume is 0.000000
-Mesh Surface is 0.000019
-Thin shell barycenter -0.002534 -0.000000 0.000450
-Center of Mass is -0.002534 -0.000000 0.000450
-Inertia Tensor is :
-| 0.000000 -0.000000 -0.000000 |
-| -0.000000 0.000000 -0.000000 |
-| -0.000000 -0.000000 0.000000 |
-Principal axes are :
-| 1.000000 -0.000000 0.000009 |
-| -0.000000 0.998526 0.054276 |
-| -0.000009 -0.054276 0.998526 |
-axis momenta are :
-| 0.000000 0.000000 0.000000 | -->
   <link name="wheel_right_link" type="wheel">
      <inertial>
@@ -142,5 +81,5 @@
 	<origin xyz="0 0 0" rpy="0 0 -1.57" />
 	<geometry>
-	 <mesh filename="package://neo_mp_500/robot_model/mp_500/meshes/MP500-WHEEL.STL" scale="0.01 0.01 0.01" />
+	 <mesh filename="package://mp500_description/meshes/MP500-WHEEL.STL" scale="0.01 0.01 0.01" />
 	</geometry>
 	<material name="Neobotix/Black" />
@@ -155,5 +94,5 @@
 <!--+++++++++++++++++++wheel_right_joint++++++++++++++++++++++++-->
    <joint name="wheel_right_joint" type="revolute">
-     <origin xyz="-0.155 -0.255 0.13" rpy="0 0 0" />
+     <origin xyz="0 -0.255 0.13" rpy="0 0 0" />
     	<axis xyz="0 1 0"/>
     	<limit effort="10000.0" lower="-1e+16" upper="1e+16" velocity="11.6"/>
@@ -162,140 +101,4 @@
     	<child link="wheel_right_link" />
     </joint>
-<!--+++++++++++++++++++laserscanner_front_joint++++++++++++++++++++++++-->
-   <joint name="laserscanner_front_joint" type="fixed">
-     <axis xyz="0 0 1" />
-     <origin xyz="-0.39 0 0.281" rpy="0 0 0" />
-     <parent link="base_link"/>
-     <child link="laserscanner_front_link"/>
-   </joint>
-<!--+++++++++++++++++++laserscanner_front_link++++++++++++++++++++++++-->
-   <link name="laserscanner_front_link" type="laser">
-	<inertial>
-		<mass value="0.01" />
-		<origin xyz="0 0 0" rpy="3.14 0 -1.57" />
-		<inertia ixx="0.001" ixy="0" ixz="0" iyy="0.001" iyz="0" izz="0.001" />
-        </inertial>
- 	<visual>
-		<origin xyz="0 0 -0.04" rpy="3.14 0 -1.57" />
-		<geometry>
-                            <!--cylinder length="0.154" radius="0.053" /-->
-                     <mesh filename="package://neo_mp_500/robot_model/mp_500/meshes/SICK-S300.STL" />
-		</geometry>
-		<material name="Neobotix/Yellow" />
-  	</visual>
-  	<collision>
-		<origin xyz="0 0 0" rpy="3.14 0 -1.57" />
-		<geometry>
-	  	<cylinder length="0.154" radius="0.053" />
-		</geometry>
-  	</collision>
-   </link>
-<!--+++++++++++++++ wheel_hanger+++++++++++++++++++++++++++-->
-   <link name="hanger">
-      <inertial>
-		  <mass value="0.01" />
-		  <origin xyz="0 0 0" rpy="0 0 0" />
-		  <inertia ixx="0.0013" ixy="0" ixz="0" iyy="0.0013" iyz="0" izz="0.0013" />
-      </inertial>
-      <visual>
-	<origin xyz="0 0 0" rpy="0 0 -1.57" />
-	<geometry>
-	      <mesh filename="package://neo_mp_500/robot_model/mp_500/meshes/HANGER-WHEEL.STL" scale="0.01 0.01 0.01" />
-	 </geometry>
-	 <material name="Neobotix/Grey" />
-	</visual>
-       <collision>
-		 <origin xyz="0 0 0" rpy="0 0 -1.57" />
-		 <geometry>
-          	 <sphere radius="0.00115"/>
-		 </geometry>
-       </collision>
-   </link>
-   <joint name="hanger_joint" type="fixed">
-    	<origin xyz="0.255 0 0.11" rpy="0 0 0"/>
-    	<axis xyz="0 0 1"/>
-    	<limit effort="10000.0" lower="-1e+16" upper="1e+16" velocity="13.5"/>
-    	<joint_properties damping="0.0" friction="0.0" />
-    	<parent link="base_link" />
-    	<child link="hanger" />
-   </joint>
-<!--+++++++++++++++ castor_front +++++++++++++++++++++++++++-->
-   <link name="castor_front">
-	<inertial>
-	  <mass value="0.25" />
-	  <origin xyz="0 0 0" rpy="0 0 0" />
-	  <inertia ixx="0.000025" ixy="0" ixz="0" iyy="0.000025" iyz="0" izz="0.000025" />
-	</inertial>
-	<visual>
-	  <origin xyz="0 0 0" rpy="0 0 0" />
-	  <geometry>
-            <sphere radius="0.005"/>
-	  </geometry>
-	 <material name="Neobotix/Grey" />
-	</visual>
-        <collision>
-	  <origin xyz="0 0 0" rpy="0 0 0" />
-	  <geometry>
-             <sphere radius="0.005"/>
-	  </geometry>
-	</collision>
-    </link>
-   <gazebo reference="caster_front">
-            <mu1 value="0.001" />
-            <mu2 value="0.001" />
-            <kp  value="1.0" />
-            <kd  value="1.0" />
-   </gazebo>
-   <joint name="castor_front_joint" type="fixed">
-    	<origin xyz="0.48 0 0.01" rpy="0 0 0"/>
-    	<axis xyz="0 0 1"/>
-    	<!--limit effort="100.0" velocity="13.5"/>
-    	<joint_properties damping="0.0" friction="0.0" /-->
-    	<parent link="base_link" />
-    	<child link="castor_front" />
-    </joint>
-<!--+++++++++++++++ castor_back +++++++++++++++++++++++++++-->
-   <link name="castor_back">
-	<inertial>
-	  <mass value="0.25" />
-	  <origin xyz="0 0 0" rpy="0 0 0" />
-	  <inertia ixx="0.000025" ixy="0" ixz="0" iyy="0.000025" iyz="0" izz="0.000025" />
-	</inertial>
-       <visual>
-         <origin xyz="0 0 0" rpy="0 0 0" />
-          <geometry>
-	    <sphere radius="0.005"/>
-	 </geometry>
-	 <material name="Neobotix/Grey" />
-       </visual>
-       <collision>
-	 <origin xyz="0 0 0" rpy="0 0 0" />
-	 <geometry>
-           <sphere radius="0.005"/>
-	 </geometry>
-       </collision>
-    </link>
-  <gazebo reference="caster_back">
-            <mu1 value="0.001" />
-            <mu2 value="0.001" />
-            <kp  value="1.0" />
-            <kd  value="1.0" />
-  </gazebo>
-   <joint name="castor_back_joint" type="fixed">
-    	<origin xyz="-0.21 0 0.01" rpy="0 0 0"/>
-    	<axis xyz="0 0 1"/>
-    	<!--limit effort="100.0" velocity="13.5"/>
-    	<joint_properties damping="0.0" friction="0.0" /-->
-    	<parent link="base_link" />
-    	<child link="castor_back" />
-    </joint>
-  <!--xacro:include filename="$(find schunk_description)/urdf/common.xacro" /-->
-  <!--xacro:include filename="$(find schunk_description)/urdf/materials.urdf.xacro" /-->
-  <!-- schunk lwa4d -->
-  <!--xacro:include filename="$(find schunk_description)/urdf/lwa4d/lwa4d.urdf.xacro" /-->
-  <!--xacro:include filename="$(find schunk_description)/urdf/common.xacro" /-->
-  <!--xacro:include filename="$(find schunk_description)/urdf/lwa4d/lwa4d.gazebo.xacro"/-->
-  <!--xacro:include filename="$(find schunk_description)/urdf/lwa4d/lwa4d.transmission.xacro"/-->
-  <!-- joint between base_link and lwa4p_extended_connector_link -->
 <transmission name="wheel_left_trans">
     <type>transmission_interface/SimpleTransmission</type>
@@ -305,5 +108,5 @@
     <actuator name="wheel_left_motor">
       <hardwareInterface>hardware_interface/EffortJointInterface</hardwareInterface>
-      <mechanicalReduction>0.1</mechanicalReduction>
+      <mechanicalReduction>0.09</mechanicalReduction>
     </actuator>
   </transmission>
@@ -315,5 +118,5 @@
     <actuator name="wheel_right_motor">
       <hardwareInterface>hardware_interface/EffortJointInterface</hardwareInterface>
-      <mechanicalReduction>0.1</mechanicalReduction>
+      <mechanicalReduction>0.09</mechanicalReduction>
     </actuator>
   </transmission>
